File: Hardware/Armboard/Armboard01.sch (KiCad schematic (older format))
At the start: 15 parts

Commit message: Added empty heirarchical sheets
Parts:
- renumbered .1uF to .1uF?, 10uF to 10uF?, 47uF to 47uF?, C8 to C?, C7 to C?
Changed lines of the file:
@@
 $Descr A4 11693 8268
 encoding utf-8
-Sheet 3 8
+Sheet 3 3
 Title ""
 Date ""
@@
 $EndDescr
 $Comp
-L Device:C .1uF
+L Device:C .1uF?
 U 1 1 5F67AED3
 P 7180 3890
-F 0 ".1uF" H 7295 3936 50  0000 L CNN
+F 0 ".1uF?" H 7295 3936 50  0000 L CNN
 F 1 "C1" H 7295 3845 50  0000 L CNN
 F 2 "" H 7218 3740 50  0001 C CNN
@@
 $EndComp
 $Comp
-L Device:C 10uF
+L Device:C 10uF?
 U 1 1 5F67B379
 P 7580 3890
-F 0 "10uF" H 7695 3936 50  0000 L CNN
+F 0 "10uF?" H 7695 3936 50  0000 L CNN
 F 1 "C2" H 7695 3845 50  0000 L CNN
 F 2 "" H 7618 3740 50  0001 C CNN
@@
 $EndComp
 $Comp
-L Device:C 10uF
+L Device:C 10uF?
 U 1 1 5F67B840
 P 7980 3890
-F 0 "10uF" H 8095 3936 50  0000 L CNN
+F 0 "10uF?" H 8095 3936 50  0000 L CNN
 F 1 "C3" H 8095 3845 50  0000 L CNN
 F 2 "" H 8018 3740 50  0001 C CNN
@@
 $EndComp
 $Comp
-L Device:C 10uF
+L Device:C 10uF?
 U 1 1 5F67BE7A
 P 8380 3890
-F 0 "10uF" H 8495 3936 50  0000 L CNN
+F 0 "10uF?" H 8495 3936 50  0000 L CNN
 F 1 "C4" H 8495 3845 50  0000 L CNN
 F 2 "" H 8418 3740 50  0001 C CNN
@@
 $EndComp
 $Comp
-L Device:C 10uF
+L Device:C 10uF?
 U 1 1 5F67C26D
 P 8780 3890
-F 0 "10uF" H 8895 3936 50  0000 L CNN
+F 0 "10uF?" H 8895 3936 50  0000 L CNN
 F 1 "C5" H 8895 3845 50  0000 L CNN
 F 2 "" H 8818 3740 50  0001 C CNN
@@
 $EndComp
 $Comp
-L Device:CP1 47uF
+L Device:CP1 47uF?
 U 1 1 5F67C954
 P 9180 3890
-F 0 "47uF" H 9295 3936 50  0000 L CNN
+F 0 "47uF?" H 9295 3936 50  0000 L CNN
 F 1 "CP1" H 9295 3845 50  0000 L CNN
 F 2 "" H 9180 3890 50  0001 C CNN
@@
 $EndComp
 $Comp
-L Device:CP1 47uF
+L Device:CP1 47uF?
 U 1 1 5F67D4A0
 P 9580 3890
-F 0 "47uF" H 9695 3936 50  0000 L CNN
+F 0 "47uF?" H 9695 3936 50  0000 L CNN
 F 1 "CP2" H 9695 3845 50  0000 L CNN
 F 2 "" H 9580 3890 50  0001 C CNN
@@
 	2850 3700 2850 3500
 $Comp
-L Device:C C8
+L Device:C C?
 U 1 1 5F750C41
 P 3800 4050
-F 0 "C8" H 3915 4096 50  0000 L CNN
+F 0 "C?" H 3915 4096 50  0000 L CNN
 F 1 "1000uF" H 3915 4005 50  0000 L CNN
 F 2 "" H 3838 3900 50  0001 C CNN
@@
 $EndComp
 $Comp
-L Device:C C7
+L Device:C C?
 U 1 1 5F75145E
 P 3200 3500
-F 0 "C7" V 3450 3450 50  0000 L CNN
+F 0 "C?" V 3450 3450 50  0000 L CNN
 F 1 "100uF" V 3350 3400 50  0000 L CNN
 F 2 "" H 3238 3350 50  0001 C CNN
