File: Hardware/Armboard/Armboard03.sch (KiCad schematic (older format))
At the start: 0 parts

Commit message: Added TIVA Device and changed page sizes
Parts:
- added U? (x8): TM4C129E_Launchpad, symbol MRDT_Shields:TM4C129E_Launchpad
Changed lines of the file:
@@
 EELAYER 30 0
 EELAYER END
-$Descr A4 11693 8268
+$Descr A 11000 8500
 encoding utf-8
-Sheet 1 9
+Sheet 4 9
 Title ""
 Date ""
@@
 Comment4 ""
 $EndDescr
+$Comp
+L MRDT_Shields:TM4C129E_Launchpad U?
+U 1 1 5F752485
+P 3810 3400
+F 0 "U?" H 3830 4670 60  0000 L CNN
+F 1 "TM4C129E_Launchpad" H 3020 4560 60  0000 L CNN
+F 2 "" H 3810 3400 60  0001 C CNN
+F 3 "" H 3810 3400 60  0001 C CNN
+	1    3810 3400
+	1    0    0    -1
+$EndComp
+$Comp
+L MRDT_Shields:TM4C129E_Launchpad U?
+U 2 1 5F752EEB
+P 4310 3400
+F 0 "U?" H 4430 4690 60  0000 C CNN
+F 1 "TM4C129E_Launchpad" H 4030 4570 60  0000 C CNN
+F 2 "" H 4310 3400 60  0001 C CNN
+F 3 "" H 4310 3400 60  0001 C CNN
+	2    4310 3400
+	-1   0    0    -1
+$EndComp
+$Comp
+L MRDT_Shields:TM4C129E_Launchpad U?
+U 3 1 5F753E3C
+P 3800 5520
+F 0 "U?" H 3860 6820 60  0000 L CNN
+F 1 "TM4C129E_Launchpad" H 3050 6710 60  0000 L CNN
+F 2 "" H 3800 5520 60  0001 C CNN
+F 3 "" H 3800 5520 60  0001 C CNN
+	3    3800 5520
+	1    0    0    -1
+$EndComp
+$Comp
+L MRDT_Shields:TM4C129E_Launchpad U?
+U 4 1 5F754D60
+P 4300 5520
+F 0 "U?" H 4460 6800 60  0000 C CNN
+F 1 "TM4C129E_Launchpad" H 4050 6680 60  0000 C CNN
+F 2 "" H 4300 5520 60  0001 C CNN
+F 3 "" H 4300 5520 60  0001 C CNN
+	4    4300 5520
+	-1   0    0    -1
+$EndComp
+$Comp
+L MRDT_Shields:TM4C129E_Launchpad U?
+U 5 1 5F755C93
+P 6400 3390
+F 0 "U?" H 6460 4660 60  0000 L CNN
+F 1 "TM4C129E_Launchpad" H 5650 4550 60  0000 L CNN
+F 2 "" H 6400 3390 60  0001 C CNN
+F 3 "" H 6400 3390 60  0001 C CNN
+	5    6400 3390
+	1    0    0    -1
+$EndComp
+$Comp
+L MRDT_Shields:TM4C129E_Launchpad U?
+U 6 1 5F7570A2
+P 6900 3390
+F 0 "U?" H 7060 4670 60  0000 C CNN
+F 1 "TM4C129E_Launchpad" H 6650 4560 60  0000 C CNN
+F 2 "" H 6900 3390 60  0001 C CNN
+F 3 "" H 6900 3390 60  0001 C CNN
+	6    6900 3390
+	-1   0    0    -1
+$EndComp
+$Comp
+L MRDT_Shields:TM4C129E_Launchpad U?
+U 7 1 5F757FE4
+P 6420 5520
+F 0 "U?" H 6480 6800 60  0000 L CNN
+F 1 "TM4C129E_Launchpad" H 5670 6690 60  0000 L CNN
+F 2 "" H 6420 5520 60  0001 C CNN
+F 3 "" H 6420 5520 60  0001 C CNN
+	7    6420 5520
+	1    0    0    -1
+$EndComp
+$Comp
+L MRDT_Shields:TM4C129E_Launchpad U?
+U 8 1 5F7598C0
+P 6920 5520
+F 0 "U?" H 7090 6810 60  0000 C CNN
+F 1 "TM4C129E_Launchpad" H 6680 6690 60  0000 C CNN
+F 2 "" H 6920 5520 60  0001 C CNN
+F 3 "" H 6920 5520 60  0001 C CNN
+	8    6920 5520
+	-1   0    0    -1
+$EndComp
 $EndSCHEMATC
