File: Hardware/Armboard/Armboard08.sch (KiCad schematic (older format))
At the start: 15 parts

Commit message: Fixed some library issues and moved Gerbs to Manufacturing folder
Parts:
- D28, D29, D30, D31, D32, D33: footprint LED_SMD:LED_0603_1608Metric_Pad1.05x0.95mm_HandSolder -> Diode_SMD:D_0603_1608Metric_Pad1.05x0.95mm_HandSolder
- R34, R35, R36, R37, R38, R39: footprint Resistor_SMD:R_0603_1608Metric_Pad1.05x0.95mm_HandSolder -> Resistor_SMD:R_0603_1608Metric_Pad0.98x0.95mm_HandSolder
Changed lines of the file:
@@
 EESchema Schematic File Version 4
+LIBS:Armboard-cache
 EELAYER 30 0
 EELAYER END
@@
 F 0 "R35" H 2870 4046 50  0000 L CNN
 F 1 "330" H 2870 3955 50  0000 L CNN
-F 2 "Resistor_SMD:R_0603_1608Metric_Pad1.05x0.95mm_HandSolder" V 2730 4000 50  0001 C CNN
+F 2 "Resistor_SMD:R_0603_1608Metric_Pad0.98x0.95mm_HandSolder" V 2730 4000 50  0001 C CNN
 F 3 "~" H 2800 4000 50  0001 C CNN
 	1    2800 4000
@@
 F 0 "D29" V 2839 4282 50  0000 R CNN
 F 1 "LED" V 2748 4282 50  0000 R CNN
-F 2 "LED_SMD:LED_0603_1608Metric_Pad1.05x0.95mm_HandSolder" H 2800 4400 50  0001 C CNN
+F 2 "Diode_SMD:D_0603_1608Metric_Pad1.05x0.95mm_HandSolder" H 2800 4400 50  0001 C CNN
 F 3 "~" H 2800 4400 50  0001 C CNN
 	1    2800 4400
@@
 F 0 "R37" H 5520 4046 50  0000 L CNN
 F 1 "330" H 5520 3955 50  0000 L CNN
-F 2 "Resistor_SMD:R_0603_1608Metric_Pad1.05x0.95mm_HandSolder" V 5380 4000 50  0001 C CNN
+F 2 "Resistor_SMD:R_0603_1608Metric_Pad0.98x0.95mm_HandSolder" V 5380 4000 50  0001 C CNN
 F 3 "~" H 5450 4000 50  0001 C CNN
 	1    5450 4000
@@
 F 0 "D31" V 5489 4282 50  0000 R CNN
 F 1 "LED" V 5398 4282 50  0000 R CNN
-F 2 "LED_SMD:LED_0603_1608Metric_Pad1.05x0.95mm_HandSolder" H 5450 4400 50  0001 C CNN
+F 2 "Diode_SMD:D_0603_1608Metric_Pad1.05x0.95mm_HandSolder" H 5450 4400 50  0001 C CNN
 F 3 "~" H 5450 4400 50  0001 C CNN
 	1    5450 4400
@@
 F 0 "R39" H 8120 4046 50  0000 L CNN
 F 1 "330" H 8120 3955 50  0000 L CNN
-F 2 "Resistor_SMD:R_0603_1608Metric_Pad1.05x0.95mm_HandSolder" V 7980 4000 50  0001 C CNN
+F 2 "Resistor_SMD:R_0603_1608Metric_Pad0.98x0.95mm_HandSolder" V 7980 4000 50  0001 C CNN
 F 3 "~" H 8050 4000 50  0001 C CNN
 	1    8050 4000
@@
 F 0 "D33" V 8089 4282 50  0000 R CNN
 F 1 "LED" V 7998 4282 50  0000 R CNN
-F 2 "LED_SMD:LED_0603_1608Metric_Pad1.05x0.95mm_HandSolder" H 8050 4400 50  0001 C CNN
+F 2 "Diode_SMD:D_0603_1608Metric_Pad1.05x0.95mm_HandSolder" H 8050 4400 50  0001 C CNN
 F 3 "~" H 8050 4400 50  0001 C CNN
 	1    8050 4400
@@
 F 0 "D28" V 2747 2975 50  0000 L CNN
 F 1 "LED" V 2838 2975 50  0000 L CNN
-F 2 "LED_SMD:LED_0603_1608Metric_Pad1.05x0.95mm_HandSolder" H 2800 2895 50  0001 C CNN
+F 2 "Diode_SMD:D_0603_1608Metric_Pad1.05x0.95mm_HandSolder" H 2800 2895 50  0001 C CNN
 F 3 "~" H 2800 2895 50  0001 C CNN
 	1    2800 2895
@@
 F 0 "R34" H 2870 3331 50  0000 L CNN
 F 1 "330" H 2870 3240 50  0000 L CNN
-F 2 "Resistor_SMD:R_0603_1608Metric_Pad1.05x0.95mm_HandSolder" V 2730 3285 50  0001 C CNN
+F 2 "Resistor_SMD:R_0603_1608Metric_Pad0.98x0.95mm_HandSolder" V 2730 3285 50  0001 C CNN
 F 3 "~" H 2800 3285 50  0001 C CNN
 	1    2800 3285
@@
 F 0 "D32" V 7997 2970 50  0000 L CNN
 F 1 "LED" V 8088 2970 50  0000 L CNN
-F 2 "LED_SMD:LED_0603_1608Metric_Pad1.05x0.95mm_HandSolder" H 8050 2890 50  0001 C CNN
+F 2 "Diode_SMD:D_0603_1608Metric_Pad1.05x0.95mm_HandSolder" H 8050 2890 50  0001 C CNN
 F 3 "~" H 8050 2890 50  0001 C CNN
 	1    8050 2890
@@
 F 0 "R38" H 8120 3326 50  0000 L CNN
 F 1 "330" H 8120 3235 50  0000 L CNN
-F 2 "Resistor_SMD:R_0603_1608Metric_Pad1.05x0.95mm_HandSolder" V 7980 3280 50  0001 C CNN
+F 2 "Resistor_SMD:R_0603_1608Metric_Pad0.98x0.95mm_HandSolder" V 7980 3280 50  0001 C CNN
 F 3 "~" H 8050 3280 50  0001 C CNN
 	1    8050 3280
@@
 F 0 "R36" H 5520 3331 50  0000 L CNN
 F 1 "330" H 5520 3240 50  0000 L CNN
-F 2 "Resistor_SMD:R_0603_1608Metric_Pad1.05x0.95mm_HandSolder" V 5380 3285 50  0001 C CNN
+F 2 "Resistor_SMD:R_0603_1608Metric_Pad0.98x0.95mm_HandSolder" V 5380 3285 50  0001 C CNN
 F 3 "~" H 5450 3285 50  0001 C CNN
 	1    5450 3285
@@
 F 0 "D30" V 5397 2975 50  0000 L CNN
 F 1 "LED" V 5488 2975 50  0000 L CNN
-F 2 "LED_SMD:LED_0603_1608Metric_Pad1.05x0.95mm_HandSolder" H 5450 2895 50  0001 C CNN
+F 2 "Diode_SMD:D_0603_1608Metric_Pad1.05x0.95mm_HandSolder" H 5450 2895 50  0001 C CNN
 F 3 "~" H 5450 2895 50  0001 C CNN
 	1    5450 2895
