File: Hardware/Armboard/Armboard07.sch (KiCad schematic (older format))
At the start: 30 parts, among them SW1 SW_Push, SW2 SW_Push, SW3 SW_Push, SW4 SW_Push, SW5 SW_Push, SW6 SW_Push

Commit message: Fixed some library issues and moved Gerbs to Manufacturing folder
Parts:
- D18, D19, D20, D21, D22, D23, D24, D25, D26, D27: footprint LED_SMD:LED_0603_1608Metric_Pad1.05x0.95mm_HandSolder -> Diode_SMD:D_0603_1608Metric_Pad1.05x0.95mm_HandSolder
- R24, R25, R26, R27, R28, R29, R30, R31, R32, R33: footprint Resistor_SMD:R_0603_1608Metric_Pad1.05x0.95mm_HandSolder -> Resistor_SMD:R_0603_1608Metric_Pad0.98x0.95mm_HandSolder
Changed lines of the file:
@@
 EESchema Schematic File Version 4
+LIBS:Armboard-cache
 EELAYER 30 0
 EELAYER END
@@
 F 0 "R30" H 7020 2676 50  0000 L CNN
 F 1 "330" H 7020 2585 50  0000 L CNN
-F 2 "Resistor_SMD:R_0603_1608Metric_Pad1.05x0.95mm_HandSolder" V 6880 2630 50  0001 C CNN
+F 2 "Resistor_SMD:R_0603_1608Metric_Pad0.98x0.95mm_HandSolder" V 6880 2630 50  0001 C CNN
 F 3 "~" H 6950 2630 50  0001 C CNN
 	1    6950 2630
@@
 F 0 "D24" V 6989 2892 50  0000 R CNN
 F 1 "LED" V 6898 2892 50  0000 R CNN
-F 2 "LED_SMD:LED_0603_1608Metric_Pad1.05x0.95mm_HandSolder" H 6950 3010 50  0001 C CNN
+F 2 "Diode_SMD:D_0603_1608Metric_Pad1.05x0.95mm_HandSolder" H 6950 3010 50  0001 C CNN
 F 3 "~" H 6950 3010 50  0001 C CNN
 	1    6950 3010
@@
 F 0 "R31" H 7020 4576 50  0000 L CNN
 F 1 "330" H 7020 4485 50  0000 L CNN
-F 2 "Resistor_SMD:R_0603_1608Metric_Pad1.05x0.95mm_HandSolder" V 6880 4530 50  0001 C CNN
+F 2 "Resistor_SMD:R_0603_1608Metric_Pad0.98x0.95mm_HandSolder" V 6880 4530 50  0001 C CNN
 F 3 "~" H 6950 4530 50  0001 C CNN
 	1    6950 4530
@@
 F 0 "D25" V 6989 4792 50  0000 R CNN
 F 1 "LED" V 6898 4792 50  0000 R CNN
-F 2 "LED_SMD:LED_0603_1608Metric_Pad1.05x0.95mm_HandSolder" H 6950 4910 50  0001 C CNN
+F 2 "Diode_SMD:D_0603_1608Metric_Pad1.05x0.95mm_HandSolder" H 6950 4910 50  0001 C CNN
 F 3 "~" H 6950 4910 50  0001 C CNN
 	1    6950 4910
@@
 F 0 "R32" H 8980 2706 50  0000 L CNN
 F 1 "330" H 8980 2615 50  0000 L CNN
-F 2 "Resistor_SMD:R_0603_1608Metric_Pad1.05x0.95mm_HandSolder" V 8840 2660 50  0001 C CNN
+F 2 "Resistor_SMD:R_0603_1608Metric_Pad0.98x0.95mm_HandSolder" V 8840 2660 50  0001 C CNN
 F 3 "~" H 8910 2660 50  0001 C CNN
 	1    8910 2660
@@
 F 0 "D26" V 8949 2922 50  0000 R CNN
 F 1 "LED" V 8858 2922 50  0000 R CNN
-F 2 "LED_SMD:LED_0603_1608Metric_Pad1.05x0.95mm_HandSolder" H 8910 3040 50  0001 C CNN
+F 2 "Diode_SMD:D_0603_1608Metric_Pad1.05x0.95mm_HandSolder" H 8910 3040 50  0001 C CNN
 F 3 "~" H 8910 3040 50  0001 C CNN
 	1    8910 3040
@@
 F 0 "R33" H 8980 4606 50  0000 L CNN
 F 1 "330" H 8980 4515 50  0000 L CNN
-F 2 "Resistor_SMD:R_0603_1608Metric_Pad1.05x0.95mm_HandSolder" V 8840 4560 50  0001 C CNN
+F 2 "Resistor_SMD:R_0603_1608Metric_Pad0.98x0.95mm_HandSolder" V 8840 4560 50  0001 C CNN
 F 3 "~" H 8910 4560 50  0001 C CNN
 	1    8910 4560
@@
 F 0 "D27" V 8949 4822 50  0000 R CNN
 F 1 "LED" V 8858 4822 50  0000 R CNN
-F 2 "LED_SMD:LED_0603_1608Metric_Pad1.05x0.95mm_HandSolder" H 8910 4940 50  0001 C CNN
+F 2 "Diode_SMD:D_0603_1608Metric_Pad1.05x0.95mm_HandSolder" H 8910 4940 50  0001 C CNN
 F 3 "~" H 8910 4940 50  0001 C CNN
 	1    8910 4940
@@
 F 0 "R24" V 2843 1750 50  0000 C CNN
 F 1 "330" V 2934 1750 50  0000 C CNN
-F 2 "Resistor_SMD:R_0603_1608Metric_Pad1.05x0.95mm_HandSolder" V 2980 1750 50  0001 C CNN
+F 2 "Resistor_SMD:R_0603_1608Metric_Pad0.98x0.95mm_HandSolder" V 2980 1750 50  0001 C CNN
 F 3 "~" H 3050 1750 50  0001 C CNN
 	1    3050 1750
@@
 F 0 "R25" V 2843 2700 50  0000 C CNN
 F 1 "330" V 2934 2700 50  0000 C CNN
-F 2 "Resistor_SMD:R_0603_1608Metric_Pad1.05x0.95mm_HandSolder" V 2980 2700 50  0001 C CNN
+F 2 "Resistor_SMD:R_0603_1608Metric_Pad0.98x0.95mm_HandSolder" V 2980 2700 50  0001 C CNN
 F 3 "~" H 3050 2700 50  0001 C CNN
 	1    3050 2700
@@
 F 0 "R26" V 2843 3650 50  0000 C CNN
 F 1 "330" V 2934 3650 50  0000 C CNN
-F 2 "Resistor_SMD:R_0603_1608Metric_Pad1.05x0.95mm_HandSolder" V 2980 3650 50  0001 C CNN
+F 2 "Resistor_SMD:R_0603_1608Metric_Pad0.98x0.95mm_HandSolder" V 2980 3650 50  0001 C CNN
 F 3 "~" H 3050 3650 50  0001 C CNN
 	1    3050 3650
@@
 F 0 "R27" V 2843 4650 50  0000 C CNN
 F 1 "330" V 2934 4650 50  0000 C CNN
-F 2 "Resistor_SMD:R_0603_1608Metric_Pad1.05x0.95mm_HandSolder" V 2980 4650 50  0001 C CNN
+F 2 "Resistor_SMD:R_0603_1608Metric_Pad0.98x0.95mm_HandSolder" V 2980 4650 50  0001 C CNN
 F 3 "~" H 3050 4650 50  0001 C CNN
 	1    3050 4650
@@
 F 0 "R28" V 2843 5600 50  0000 C CNN
 F 1 "330" V 2934 5600 50  0000 C CNN
-F 2 "Resistor_SMD:R_0603_1608Metric_Pad1.05x0.95mm_HandSolder" V 2980 5600 50  0001 C CNN
+F 2 "Resistor_SMD:R_0603_1608Metric_Pad0.98x0.95mm_HandSolder" V 2980 5600 50  0001 C CNN
 F 3 "~" H 3050 5600 50  0001 C CNN
 	1    3050 5600
@@
 F 0 "R29" V 2843 6550 50  0000 C CNN
 F 1 "330" V 2934 6550 50  0000 C CNN
-F 2 "Resistor_SMD:R_0603_1608Metric_Pad1.05x0.95mm_HandSolder" V 2980 6550 50  0001 C CNN
+F 2 "Resistor_SMD:R_0603_1608Metric_Pad0.98x0.95mm_HandSolder" V 2980 6550 50  0001 C CNN
 F 3 "~" H 3050 6550 50  0001 C CNN
 	1    3050 6550
@@
 F 0 "D18" H 3493 1495 50  0000 C CNN
 F 1 "LED" H 3493 1586 50  0000 C CNN
-F 2 "LED_SMD:LED_0603_1608Metric_Pad1.05x0.95mm_HandSolder" H 3500 1750 50  0001 C CNN
+F 2 "Diode_SMD:D_0603_1608Metric_Pad1.05x0.95mm_HandSolder" H 3500 1750 50  0001 C CNN
 F 3 "~" H 3500 1750 50  0001 C CNN
 	1    3500 1750
@@
 F 0 "D19" H 3493 2445 50  0000 C CNN
 F 1 "LED" H 3493 2536 50  0000 C CNN
-F 2 "LED_SMD:LED_0603_1608Metric_Pad1.05x0.95mm_HandSolder" H 3500 2700 50  0001 C CNN
+F 2 "Diode_SMD:D_0603_1608Metric_Pad1.05x0.95mm_HandSolder" H 3500 2700 50  0001 C CNN
 F 3 "~" H 3500 2700 50  0001 C CNN
 	1    3500 2700
@@
 F 0 "D20" H 3493 3395 50  0000 C CNN
 F 1 "LED" H 3493 3486 50  0000 C CNN
-F 2 "LED_SMD:LED_0603_1608Metric_Pad1.05x0.95mm_HandSolder" H 3500 3650 50  0001 C CNN
+F 2 "Diode_SMD:D_0603_1608Metric_Pad1.05x0.95mm_HandSolder" H 3500 3650 50  0001 C CNN
 F 3 "~" H 3500 3650 50  0001 C CNN
 	1    3500 3650
@@
 F 0 "D21" H 3493 4395 50  0000 C CNN
 F 1 "LED" H 3493 4486 50  0000 C CNN
-F 2 "LED_SMD:LED_0603_1608Metric_Pad1.05x0.95mm_HandSolder" H 3500 4650 50  0001 C CNN
+F 2 "Diode_SMD:D_0603_1608Metric_Pad1.05x0.95mm_HandSolder" H 3500 4650 50  0001 C CNN
 F 3 "~" H 3500 4650 50  0001 C CNN
 	1    3500 4650
@@
 F 0 "D22" H 3493 5345 50  0000 C CNN
 F 1 "LED" H 3493 5436 50  0000 C CNN
-F 2 "LED_SMD:LED_0603_1608Metric_Pad1.05x0.95mm_HandSolder" H 3500 5600 50  0001 C CNN
+F 2 "Diode_SMD:D_0603_1608Metric_Pad1.05x0.95mm_HandSolder" H 3500 5600 50  0001 C CNN
 F 3 "~" H 3500 5600 50  0001 C CNN
 	1    3500 5600
@@
 F 0 "D23" H 3493 6295 50  0000 C CNN
 F 1 "LED" H 3493 6386 50  0000 C CNN
-F 2 "LED_SMD:LED_0603_1608Metric_Pad1.05x0.95mm_HandSolder" H 3500 6550 50  0001 C CNN
+F 2 "Diode_SMD:D_0603_1608Metric_Pad1.05x0.95mm_HandSolder" H 3500 6550 50  0001 C CNN
 F 3 "~" H 3500 6550 50  0001 C CNN
 	1    3500 6550
